File: alpha_board/hardware/ee110_alpha_board.kicad_sch (KiCad schematic)
At the start: 44 parts, among them J3 wall, J4 battery, J5 AVR-JTAG-10, SW1 RESET, U10 CC2652R1FRGZR, U7 LM1086, U8 LM372x, U9 LM1086, X1 Crystal_GND24, X2 Crystal_GND24

Commit message: biig progress
Parts:
- removed J3: wall, symbol Connector:Conn_01x03_Pin
- removed J4: battery, symbol Connector:Conn_01x03_Pin
- removed X2: Crystal_GND24, symbol Device:Crystal_GND24
- added B1: 1049P, My_Footprint:1049P_KEY, symbol EE110_Battery:1049P
- added C20: 1uF, Capacitor_SMD:C_0603_1608Metric, symbol Device:C_Small
- added D7: LED, Diode_SMD:D_0805_2012Metric, symbol Device:LED
- added J1: power, Connector:JWT_A3963_1x02_P3.96mm_Vertical, symbol Connector:Conn_01x02_Pin
- added L1: BLM18HE152SN1, Inductor_SMD:L_7.3x7.3_H3.5, symbol Device:L
- added R1: 1, Resistor_SMD:R_0603_1608Metric, symbol Device:R_US
- added R16: 470, Resistor_SMD:R_0603_1608Metric, symbol Device:R_US
- added X2: 32.768KHz, Crystal:Crystal_SMD_3215-2Pin_3.2x1.5mm, symbol Device:Crystal
- AE1: footprint (none) -> My_Footprint:EE110_Antenna
- C1: renamed from C2; footprint (none) -> Capacitor_Tantalum_SMD:CP_EIA-1608-08_AVX-J
- C10: renamed from C20; footprint (none) -> Capacitor_Tantalum_SMD:CP_EIA-1608-08_AVX-J
- C11: renamed from C23; footprint (none) -> Capacitor_Tantalum_SMD:CP_EIA-1608-08_AVX-J
- C12: renamed from C13; value C_Polarized_Small_US -> 5uF; footprint (none) -> Capacitor_Tantalum_SMD:CP_EIA-1608-08_AVX-J
- C13: renamed from C17; value C_Polarized_Small_US -> 5uF; footprint (none) -> Capacitor_Tantalum_SMD:CP_EIA-1608-08_AVX-J
- C14: renamed from C3; footprint (none) -> Capacitor_SMD:C_0603_1608Metric
- C15: renamed from C8; footprint (none) -> Capacitor_SMD:C_0603_1608Metric
- C16: renamed from C18; value C_Polarized_Small_US -> 5uF; footprint (none) -> Capacitor_SMD:CP_Elec_3x5.3
- C17: renamed from C4; footprint (none) -> Capacitor_SMD:C_0603_1608Metric
- C18: renamed from C21; value C_Polarized_Small_US -> 5uF; footprint (none) -> Capacitor_SMD:CP_Elec_3x5.3
- C19: renamed from C9; footprint (none) -> Capacitor_SMD:C_0603_1608Metric
- C2: renamed from C7; footprint (none) -> Capacitor_Tantalum_SMD:CP_EIA-1608-08_AVX-J
- C21: renamed from C5; footprint (none) -> Capacitor_SMD:C_0603_1608Metric
- C22: renamed from C6; footprint (none) -> Capacitor_SMD:C_0603_1608Metric
- C23: renamed from C10; footprint (none) -> Capacitor_SMD:C_0603_1608Metric
- C3: renamed from C16; footprint (none) -> Capacitor_Tantalum_SMD:CP_EIA-1608-08_AVX-J
- C4: renamed from C11; footprint (none) -> Capacitor_Tantalum_SMD:CP_EIA-1608-08_AVX-J
- C5: renamed from C12; footprint (none) -> Capacitor_Tantalum_SMD:CP_EIA-1608-08_AVX-J
- C6: renamed from C14; footprint (none) -> Capacitor_Tantalum_SMD:CP_EIA-1608-08_AVX-J
- C7: renamed from C19; footprint (none) -> Capacitor_Tantalum_SMD:CP_EIA-1608-08_AVX-J
- C8: renamed from C22; footprint (none) -> Capacitor_Tantalum_SMD:CP_EIA-1608-08_AVX-J
- C9: renamed from C15; footprint (none) -> Capacitor_Tantalum_SMD:CP_EIA-1608-08_AVX-J
- D1: renamed from D5; footprint (none) -> Diode_SMD:D_0603_1608Metric
- D2: renamed from D6; footprint (none) -> Diode_SMD:D_0603_1608Metric
- J2: renamed from J5; footprint (none) -> My_Footprint:CON10_2X5_DUK_FTSH_SAI
- L2: renamed from L5; footprint (none) -> Inductor_SMD:L_0603_1608Metric
- L3: renamed from L1; footprint (none) -> Inductor_SMD:L_0603_1608Metric
- L4: footprint (none) -> Inductor_SMD:L_0603_1608Metric
- L5: renamed from L2; footprint (none) -> Inductor_SMD:L_0603_1608Metric
- L6: renamed from L3; footprint (none) -> Inductor_SMD:L_0603_1608Metric
- R2: renamed from R4; footprint (none) -> Resistor_SMD:R_0603_1608Metric
- R3: renamed from R6; footprint (none) -> Resistor_SMD:R_0603_1608Metric
- R4: renamed from R3; footprint (none) -> Resistor_SMD:R_0603_1608Metric
- R5: footprint (none) -> Resistor_SMD:R_0603_1608Metric
- SW1: footprint (none) -> Button_Switch_THT:SW_PUSH_6mm
- U1: renamed from U10; footprint RGZ0048A -> My_Footprint:RGZ0048A_NV
- U2: renamed from U8; footprint (none) -> Package_TO_SOT_SMD:SOT-23-5
- U3: renamed from U7; footprint (none) -> Package_TO_SOT_SMD:TO-263-3_TabPin2
- U4: renamed from U9; footprint (none) -> Package_TO_SOT_SMD:TO-263-3_TabPin2
- X1: value Crystal_GND24 -> 48MHz; footprint (none) -> Crystal:Crystal_SMD_2016-4Pin_2.0x1.6mm
Connections:
- net +3.3V: now also U2.5 (Vcc), L1.1, R1.2; no longer C3.1, C4.1, C5.1, C6.1, C7.1, C8.1, R3.1, U1.13 (VDDS2), U1.22 (VDDS3), U1.34 (VDDS_DCDC), U1.44 (VDDS), U2. (Vcc), U4.2 (VO)
- net +5V: now also R16.1; no longer C1.1, U3.3 (VI)
- net GND: now also B1.2, C20.2, D7.1 (K), J1.2 (Pin_2); no longer U2. (Vcc)
- net at SW1.2: now also U2.4 (MR); no longer U2. (Vcc)
- net at U1.23 (DCOUPL): now also C20.1
- net at C16.1, U1.3 (X32K_Q1): now also X2.2
- net at U1.35 (RESET_N): now also J2.6 (~{SRST}), U2.3 (RESET); no longer U2. (Vcc)
- net at C18.1, U1.4 (X32K_Q2): now also X2.1
- net gpio/DIO_0 renamed gpio/LCD_DATA0
- net gpio/DIO_1 renamed gpio/LCD_DATA1
- net gpio/DIO_10 renamed gpio/LCD_RS
- net gpio/DIO_11 renamed gpio/SPI_MOSI
- net gpio/DIO_12 renamed gpio/SPI_MISO
- net gpio/DIO_13 renamed gpio/SPI_SCLK
- net gpio/DIO_14 renamed gpio/IMU_CS
- net gpio/DIO_15 renamed gpio/SD_CS
- net gpio/DIO_16 renamed gpio/KEYPAD_ROWA
- net gpio/DIO_17 renamed gpio/KEYPAD_ROWB
- net gpio/DIO_18 renamed gpio/KEYPAD_COL1
- net gpio/DIO_19 renamed gpio/KEYPAD_COL2
- net gpio/DIO_2 renamed gpio/LCD_DATA2
- net gpio/DIO_20 renamed gpio/KEYPAD_COL3
- net gpio/DIO_21 renamed gpio/KEYPAD_COL4
- net gpio/DIO_22 renamed gpio/TEST
- net gpio/DIO_23 renamed gpio/VBAT_READ
- net gpio/DIO_24 renamed gpio/SERVO1_PWM
- net gpio/DIO_25 renamed gpio/SERVO2_PWM
- net gpio/DIO_26 renamed gpio/SERVO1_POS
- net gpio/DIO_27 renamed gpio/SERVO2_POS
- net gpio/DIO_28 renamed gpio/SPKR
- net gpio/DIO_29: no longer names the net of U1.42 (DIO_29)
- net gpio/DIO_3 renamed gpio/LCD_DATA3
- net gpio/DIO_30: no longer names the net of U1.43 (DIO_30)
- net gpio/DIO_4 renamed gpio/LCD_DATA4
- net gpio/DIO_5 renamed gpio/LCD_DATA5
- net gpio/DIO_6 renamed gpio/LCD_DATA6
- net gpio/DIO_7 renamed gpio/LCD_DATA7
- net gpio/DIO_8 renamed gpio/LCD_E
- net gpio/DIO_9 renamed gpio/LCD_RW
- new net: C4.1, C5.1, C6.1, C7.1, C8.1, L1.2, U1.13 (VDDS2), U1.22 (VDDS3), U1.34 (VDDS_DCDC), U1.44 (VDDS)
- new net: C3.1, R1.1, R3.1, U4.2 (VO)
- new net: D7.2 (A), R16.2
- new net: B1.1, B1.3
- new net +5VD: B1.4, C1.1, J1.1 (Pin_1), U3.3 (VI)
- no-connect marks 1 -> 0
Other:
- sheet gpio ports: added IMU_CS, KEYPAD_COL1, KEYPAD_COL2, KEYPAD_COL3, KEYPAD_COL4, KEYPAD_ROWA, KEYPAD_ROWB, LCD_DATA0, LCD_DATA1, LCD_DATA2, LCD_DATA3, LCD_DATA4, LCD_DATA5, LCD_DATA6, LCD_DATA7, LCD_E, LCD_RS, LCD_RW, SD_CS, SERVO1_POS, SERVO1_PWM, SERVO2_POS, SERVO2_PWM, SPI_MISO, SPI_MOSI, SPI_SCLK, SPKR, TEST, VBAT_READ; removed DIO_0, DIO_1, DIO_10, DIO_11, DIO_12, DIO_13, DIO_14, DIO_15, DIO_16, DIO_17, DIO_18, DIO_19, DIO_2, DIO_20, DIO_21, DIO_22, DIO_23, DIO_24, DIO_25, DIO_26, DIO_27, DIO_28, DIO_29, DIO_3, DIO_30, DIO_4, DIO_5, DIO_6, DIO_7, DIO_8, DIO_9
- note added: "C0G/NP0 caps"
- note added: "C_{L}=7uF"
- note added: "C_{T}=2uF"
- note added: "C_{mc}=7uF"
- note added: "Pin 13"
- note added: "Pin 22"
- note added: "Pin 34"
- note added: "Pin 44"
- note added: "Pin 45"
- note added: "Pin 48"
- note added: "RF ground"
- note added: "X5R/X7R caps"
- note added: "analog ground"
- note added: "digital ground (label omitted elsewhere)"
- note added: "power LED"
- note added: "servo ground"
- moved on the sheet: AE1, C1, C14, C15, C17, C19, C2, C21, C22, C23, C3, C4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
