File: alpha_board/hardware/ee110_alpha_board.kicad_sch (KiCad schematic)
At the start: 46 parts, among them J1 power, J2 AVR-JTAG-10, SW1 RESET, U1 LM1086, U2 LM1086, U3 LM372x, U4 CC2652R1FRGZR, X1 48MHz, X2 32.768KHz

Commit message: Ilana committing from laptop
Parts:
- C1, C10, C11, C12, C14, C16, C2, C21, C3, C4, C5, C6, C7, C8, C9: footprint Capacitor_Tantalum_SMD:CP_EIA-1608-08_AVX-J -> Capacitor_Tantalum_SMD:CP_EIA-1608-08_AVX-J_Pad1.25x1.05mm_HandSolder
- C13, C15, C17, C18, C19, C20: footprint Capacitor_SMD:C_1206_3216Metric -> Capacitor_SMD:C_1206_3216Metric_Pad1.33x1.80mm_HandSolder
- C22: footprint Capacitor_SMD:C_0603_1608Metric -> Capacitor_SMD:C_0603_1608Metric_Pad1.08x0.95mm_HandSolder
- D2, D3: footprint Diode_SMD:D_0603_1608Metric -> Diode_SMD:D_0603_1608Metric_Pad1.05x0.95mm_HandSolder
- L2: footprint Inductor_SMD:L_0603_1608Metric -> Inductor_SMD:L_0603_1608Metric_Pad1.05x0.95mm_HandSolder
- L3, L4, L5: footprint Inductor_SMD:L_1206_3216Metric -> Inductor_SMD:L_1206_3216Metric_Pad1.22x1.90mm_HandSolder
- R2, R3, R4, R5, R6: footprint Resistor_SMD:R_0603_1608Metric -> Resistor_SMD:R_0603_1608Metric_Pad0.98x0.95mm_HandSolder
Connections:
- net +3.3V: no longer R4.1
- net +5V: now also R4.1
- net gpio/SERVO1_POS: now also U4.41 (DIO_28); no longer U4.40 (DIO_27)
- net gpio/SERVO1_PWM: now also U4.43 (DIO_30); no longer U4.42 (DIO_29)
- net gpio/SERVO2_POS: now also U4.40 (DIO_27); no longer U4.39 (DIO_26)
- net gpio/SERVO2_PWM: now also U4.42 (DIO_29); no longer U4.41 (DIO_28)
- net gpio/SPKR: now also U4.38 (DIO_25); no longer U4.43 (DIO_30)
- net gpio/VBAT_READ: now also U4.39 (DIO_26); no longer U4.38 (DIO_25)
- net gpio/TEST renamed gpio/TEST_BLUE
- net gpio/TEST_LED renamed gpio/TEST_GREEN
Other:
- sheet gpio ports: added TEST_BLUE, TEST_GREEN; removed TEST, TEST_LED
- note removed: "power led"
- moved on the sheet: D1, R4
