File: alpha_board/hardware/ee110_alpha_board_gpio.kicad_sch (KiCad schematic)
At the start: 41 parts, among them J4 Micro_SD_Card, J5 4P4C, J6 4P4C, SW2 TEST_BUTTON, U5 74LS138, U6 74LVC245, U7 LM386, U8 LM2902, U9 MPU-9250

Commit message: Ilana committing from laptop
Parts:
- added D10, D11: D_Small_Filled, Diode_SMD:D_1206_3216Metric_Pad1.42x1.75mm_HandSolder, symbol Device:D_Small_Filled
- added D9: LED_BLUE, LED_SMD:LED_0603_1608Metric_Pad1.05x0.95mm_HandSolder, symbol Device:LED
- added R8: 200, Resistor_SMD:R_0603_1608Metric_Pad0.98x0.95mm_HandSolder, symbol Device:R_US
- C23, C24, C25, C26, C27, C28, C29: footprint Capacitor_SMD:C_0603_1608Metric -> Capacitor_SMD:C_0603_1608Metric_Pad1.08x0.95mm_HandSolder
- D4, D5, D6, D7: footprint Diode_SMD:D_0603_1608Metric -> Diode_SMD:D_0603_1608Metric_Pad1.05x0.95mm_HandSolder
- D8: value LED -> LED_GREEN; footprint LED_SMD:LED_0603_1608Metric -> LED_SMD:LED_0603_1608Metric_Pad1.05x0.95mm_HandSolder
- R1: renamed from R7; footprint Resistor_SMD:R_0603_1608Metric -> Resistor_SMD:R_0603_1608Metric_Pad0.98x0.95mm_HandSolder
- R10, R11, R12, R13, R14, R15, R9: footprint Resistor_SMD:R_0603_1608Metric -> Resistor_SMD:R_0603_1608Metric_Pad0.98x0.95mm_HandSolder
- R7: renamed from R8; footprint Resistor_SMD:R_0603_1608Metric -> Resistor_SMD:R_0603_1608Metric_Pad0.98x0.95mm_HandSolder
- TP2: value TEST_LED -> TEST_GREEN
- TP3: renamed from TP5; value TEST -> TEST_BLUE
- U9: footprint Sensor_Motion:InvenSense_QFN-24_3x3mm_P0.4mm -> Package_DFN_QFN:QFN-24-1EP_3x3mm_P0.4mm_EP1.75x1.6mm
- renumbered TP3 to TP4, TP4 to TP5
Connections:
- net +VBAT: now also D10.2 (A), D11.2 (A); no longer J5.4, J6.4
- net GND: now also D9.1 (K)
- net TEST renamed TEST_BLUE
- net TEST_BLUE: now also R8.2
- net TEST_LED renamed TEST_GREEN
- new net: D9.2 (A), R8.1
- new net: D11.1 (K), J6.4
- new net: D10.1 (K), J5.4
Other:
- moved on the sheet: D8, R1, R7, SW2, TP1, TP2, TP3, TP4, TP5
