File: alpha_board/hardware/ee110_alpha_board.kicad_pcb (KiCad board)
At the start: 2 copper layers, 104.1 x 144.8 mm, 85 parts, among them J1 power, J2 AVR-JTAG-10, J4 4P4C, J5 4P4C, J6 Micro_SD_Card, Q1 TIP120, SW1 RESET, U1 CC2652R1FRGZR, U11 MPU-9250, U2 LM372x, U3 LM1086, U4 LM1086, U5 74LS138, U7 74LVC245, U8 LM386, U9 LM2902, X1 48MHz, X2 32.768KHz

Commit message: first revision
Parts:
- removed C30: 0.05uF, Capacitor_SMD:C_0603_1608Metric
- removed L6: 2nH, Inductor_SMD:L_0603_1608Metric
- removed Q1: TIP120, Package_TO_SOT_THT:TO-220-3_Vertical
- removed R1: 1, Resistor_SMD:R_0603_1608Metric
- removed the R12 at (-40.7, 72.9)
- removed the R12 at (-107.8, -55.1)
- removed R16: 470, Resistor_SMD:R_0603_1608Metric
- removed U11: MPU-9250, Sensor_Motion:InvenSense_QFN-24_3x3mm_P0.4mm
- added D8: TEST_LED, LED_SMD:LED_0603_1608Metric, F.Cu at (48.5, 149.1)
- added DS1: LCD-20X4B, My_Footprint:WINSTAR-WH1604A, F.Cu at (86.4, 64.1)
- added R12: 24K, Resistor_SMD:R_0603_1608Metric, F.Cu at (126.5, 132.6)
- added R13: 36K, Resistor_SMD:R_0603_1608Metric, F.Cu at (126.5, 129.8)
- added R14: 24K, Resistor_SMD:R_0603_1608Metric, F.Cu at (126.5, 138.7)
- added R15: 36K, Resistor_SMD:R_0603_1608Metric, F.Cu at (126.6, 135.9)
- added RV3: 10k, Potentiometer_THT:Potentiometer_Bourns_3296P_Horizontal, F.Cu at (124.5, 122.9)
- added SW2: TEST_BUTTON, Button_Switch_SMD:SW_SPST_TL3342, F.Cu at (48.5, 141.5)
- added TP4: GND, TestPoint:TestPoint_THTPad_2.0x2.0mm_Drill1.0mm, F.Cu at (68.6, 143.5)
- added TP5: TEST, TestPoint:TestPoint_THTPad_2.0x2.0mm_Drill1.0mm, F.Cu at (68.6, 149.4)
- AE1: value Antenna -> Antenna_Chip
- C13: value 5uF -> 1.3pF; footprint Capacitor_Tantalum_SMD:CP_EIA-1608-08_AVX-J -> Capacitor_SMD:C_1206_3216Metric
- C14, C21: value 12pF -> 5uF; footprint Capacitor_SMD:C_0603_1608Metric -> Capacitor_Tantalum_SMD:CP_EIA-1608-08_AVX-J
- C15: value 1pF -> 1.8pF; footprint Capacitor_SMD:C_0603_1608Metric -> Capacitor_SMD:C_1206_3216Metric
- C16: footprint Capacitor_SMD:CP_Elec_3x5.3 -> Capacitor_Tantalum_SMD:CP_EIA-1608-08_AVX-J
- C17: value 1pF -> 4pF; footprint Capacitor_SMD:C_0603_1608Metric -> Capacitor_SMD:C_1206_3216Metric
- C18: value 5uF -> 4pF; footprint Capacitor_SMD:CP_Elec_3x5.3 -> Capacitor_SMD:C_1206_3216Metric
- C19: footprint Capacitor_SMD:C_0603_1608Metric -> Capacitor_SMD:C_1206_3216Metric
- C20: value 1uF -> 1.3pF; footprint Capacitor_SMD:C_0603_1608Metric -> Capacitor_SMD:C_1206_3216Metric
- C22: value 1.8oF -> 1uF
- C23: value 1pF -> 10uF
- C24: value 0.1uF -> 250uF
- C25: value 10nF -> 0.05uF
- C26: value 0.1uF -> 10uF
- C27: value 250uF -> 0.1uF
- C28: value 10uF -> 10nF
- C29: value 10uF -> 0.1uF
- D1: value D_Small_Filled -> POWER LED; footprint Diode_SMD:D_0603_1608Metric -> LED_THT:LED_D3.0mm
- D7: value LED -> D_Small_Filled; footprint Diode_SMD:D_0805_2012Metric -> Diode_SMD:D_0603_1608Metric
- J1: footprint Connector:JWT_A3963_1x02_P3.96mm_Vertical -> My_Footprint:My_Power_Connector
- J4: value 4P4C -> Micro_SD_Card; footprint Connector_JST:JST_XH_S4B-XH-A-1_1x04_P2.50mm_Horizontal -> Connector_Card:microSD_HC_Hirose_DM3D-SF
- J5: value 4P4C -> Servo1
- J6: value Micro_SD_Card -> Servo2; footprint Connector_Card:microSD_HC_Hirose_DM3D-SF -> Connector_JST:JST_XH_S4B-XH-A-1_1x04_P2.50mm_Horizontal
- L3: value 2.4nH -> 3.3nH; footprint Inductor_SMD:L_0603_1608Metric -> Inductor_SMD:L_1206_3216Metric
- L4: value 2.4nH -> 2nH; footprint Inductor_SMD:L_0603_1608Metric -> Inductor_SMD:L_1206_3216Metric
- L5: value 2nH -> 3.3nH; footprint Inductor_SMD:L_0603_1608Metric -> Inductor_SMD:L_1206_3216Metric
- LS1: footprint My_Footprint:CVS-1508_CUD -> My_Footprint:SPKR_CVS-1508
- R4: value 363 -> 200
- R5: value 183 -> 363
- R6: value 24K -> 183
- R7: value 36K -> 100
- R8: value 24K -> 200
- R9: value 36K -> 10
- RV1, RV2: footprint Potentiometer_THT:Potentiometer_Bourns_3339P_Vertical -> Potentiometer_THT:Potentiometer_Bourns_3296P_Horizontal
- SW1: footprint Button_Switch_THT:SW_PUSH_6mm -> Button_Switch_SMD:SW_SPST_TL3342
- TP1: value +3.3V -> TEST_BUTTON
- TP2: value GND -> TEST_LED
- TP3: value TEST -> +3.3V
- U1: value CC2652R1FRGZR -> LM1086; footprint My_Footprint:RGZ0048A_NV -> Package_TO_SOT_SMD:TO-263-3_TabPin2
- U2: value LM372x -> LM1086; footprint Package_TO_SOT_SMD:SOT-23-5 -> Package_TO_SOT_SMD:TO-263-3_TabPin2
- U3: value LM1086 -> LM372x; footprint Package_TO_SOT_SMD:TO-263-3_TabPin2 -> Package_TO_SOT_SMD:SOT-23-5
- U4: value LM1086 -> CC2652R1FRGZR; footprint Package_TO_SOT_SMD:TO-263-3_TabPin2 -> My_Footprint:RGZ0048A_NV
- U6: value ~ -> 74LVC245; footprint Display:LM16255 -> Package_SO:SOIC-20W_7.5x15.4mm_P1.27mm
- U7: value 74LVC245 -> LM386; footprint Package_SO:SOIC-20W_7.5x15.4mm_P1.27mm -> Package_DIP:DIP-8_W7.62mm
- U8: value LM386 -> LM2902; footprint Package_DIP:DIP-8-16_W7.62mm -> Package_SO:SOIC-14_3.9x8.7mm_P1.27mm
- U9: value LM2902 -> MPU-9250; footprint Package_SO:SOIC-14_3.9x8.7mm_P1.27mm -> Sensor_Motion:InvenSense_QFN-24_3x3mm_P0.4mm
- moved R11 294.3 mm to (114.6, 135.1)
- moved R10 293.1 mm to (113.0, 132.6)
- moved C25 292.7 mm to (116.8, 120.1), turned to -90 degrees
- moved R9 292.4 mm to (116.9, 124.5), turned to -90 degrees
- moved C24 287.6 mm to (113.3, 113.8), turned to 90 degrees
- moved C26 282.7 mm to (103.6, 122.9), turned to 90 degrees
- moved R8 269.5 mm to (55.6, 149.1)
- moved R7 259.8 mm to (55.6, 143.5)
- moved R6 258.1 mm to (76.7, 118.6), turned to 180 degrees
- moved C1 252.5 mm to (86.4, 156.2), turned to 180 degrees
- moved C2 221.7 mm to (79.9, 125.2), turned to -90 degrees
- moved L1 218.7 mm to (103.9, 104.8), turned to 90 degrees
- moved C3 212.5 mm to (76.4, 122.9), turned to 180 degrees
- moved C6 212.3 mm to (104.9, 86.1)
- moved C9 211.2 mm to (110.2, 85.3)
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Connections:
- AE1 pad 1: Net-(AE1-A) -> /RF_ANT
- B1 pad 4: +5VD -> +VBAT
- C1 pad 1: +5VD -> +VBAT
- C10 pad 1: Net-(U1-VDDR) -> Net-(U4-VDDR)
- C11 pad 1: Net-(U1-VDDR) -> Net-(U4-VDDR)
- C12 pad 1: Net-(U1-X48M_P) -> Net-(U4-X48M_P)
- C13 pad 1: Net-(U1-X48M_N) -> /RF_P
- C13 pad 2: GND -> /RF_MATCH1
- C14 pad 1: GND -> Net-(U4-X48M_N)
- C14 pad 2: Net-(C14-Pad2) -> GND
- C15 pad 1: Net-(U1-RF_N) -> /RF_MATCH2
- C15 pad 2: GND -> /RF_ANT
- C16 pad 1: Net-(U1-X32K_Q1) -> Net-(U4-X32K_Q1)
- C17 pad 1: Net-(U1-RF_P) -> /RF_MATCH1
- C17 pad 2: Net-(C17-Pad2) -> GND
- C18 pad 1: Net-(U1-X32K_Q2) -> /RF_MATCH2
- C19 pad 1: Net-(C19-Pad1) -> /RF_ANT
- C20 pad 1: Net-(U1-DCOUPL) -> /RF_N
- C21 pad 1: Net-(C21-Pad1) -> Net-(U4-X32K_Q2)
- C21 pad 2: Net-(C21-Pad2) -> GND
- C22 pad 1: Net-(C21-Pad2) -> Net-(U4-DCOUPL)
- C22 pad 2: Net-(AE1-A) -> GND
- C23 pad 1: Net-(AE1-A) -> Net-(U7-BYPASS)
- C24 pad 1: +3.3V -> Net-(C24-Pad1)
- C24 pad 2: GND -> Net-(LS1-1)
- C25 pad 1: +3.3V -> Net-(C24-Pad1)
- C25 pad 2: GND -> Net-(C25-Pad2)
- C26 pad 1: Net-(U11-REGOUT) -> Net-(C26-Pad1)
- C26 pad 2: GND -> Net-(C26-Pad2)
- C27 pad 1: Net-(C27-Pad1) -> +3.3V
- C27 pad 2: Net-(LS1-1) -> GND
- C28 pad 1: Net-(C28-Pad1) -> +3.3V
- C28 pad 2: Net-(C28-Pad2) -> GND
- C29 pad 1: Net-(U8-BYPASS) -> Net-(U9-REGOUT)
- C3 pad 1: Net-(U4-VO) -> +3.3V
- C4 pad 1: Net-(U1-VDDS) -> Net-(U4-VDDS)
- C5 pad 1: Net-(U1-VDDS) -> Net-(U4-VDDS)
- C6 pad 1: Net-(U1-VDDS) -> Net-(U4-VDDS)
- C7 pad 1: Net-(U1-VDDS) -> Net-(U4-VDDS)
- C8 pad 1: Net-(U1-VDDS) -> Net-(U4-VDDS)
- C9 pad 1: Net-(U1-VDDR) -> Net-(U4-VDDR)
- D1 pad 1: Net-(D1-K) -> GND
- D1 pad 2: /gpio/KEYPAD_ROWA -> Net-(D1-A)
- D2 pad 1: /gpio/KEYPAD_ROWB -> Net-(D2-K)
- D2 pad 2: Net-(D2-A) -> /gpio/KEYPAD_ROWA
- D3 pad 1: Net-(D3-K) -> /gpio/KEYPAD_ROWB
- D3 pad 2: unconnected-(D3-A-Pad2) -> Net-(D3-A)
- D7 pad 1: GND -> Net-(D7-K)
- J1 pad 1: +5VD -> +VBAT
- J2 pad 3: Net-(D1-K) -> Net-(D2-K)
- J2 pad 9: Net-(D2-A) -> Net-(D3-A)
- J3 pad 1: unconnected-(J3-R1-Pad1) -> Net-(D7-A)
- J3 pad 2: Net-(D4-A) -> Net-(D6-A)
- J3 pad 4: Net-(D6-A) -> Net-(D4-A)
- J4 pad 1: GND -> unconnected-(J4-DAT2-Pad1)
- J4 pad 2: Net-(J4-Pad2) -> /gpio/SD_CS
- J4 pad 3: /gpio/SERVO1_PWM -> /gpio/SPI_MOSI
- J4 pad 4: +5VD -> +3.3V
- J5 pad 3: /gpio/SERVO2_PWM -> /gpio/SERVO1_PWM
- J5 pad 4: +5VD -> +VBAT
- J6 pad 1: unconnected-(J6-DAT2-Pad1) -> GND
- J6 pad 2: /gpio/SD_CS -> Net-(J6-Pad2)
- J6 pad 3: /gpio/SPI_MOSI -> /gpio/SERVO2_PWM
- J6 pad 4: +3.3V -> +VBAT
- L1 pad 2: Net-(U1-VDDS) -> Net-(U4-VDDS)
- L2 pad 1: Net-(U1-DCDC_SW) -> Net-(U4-DCDC_SW)
- L2 pad 2: Net-(U1-VDDR) -> Net-(U4-VDDR)
- L3 pad 1: Net-(C14-Pad2) -> GND
- L3 pad 2: Net-(U1-RF_P) -> /RF_P
- L4 pad 1: Net-(C17-Pad2) -> /RF_MATCH1
- L4 pad 2: Net-(U1-RF_N) -> /RF_MATCH2
- L5 pad 1: Net-(C17-Pad2) -> /RF_N
- L5 pad 2: Net-(C19-Pad1) -> /RF_MATCH1
- R10 pad 1: Net-(J5-Pad2) -> +VBAT
- R10 pad 2: Net-(U9B-+) -> Net-(U8C-+)
- R11 pad 1: Net-(U9B-+) -> Net-(U8C-+)
- R2 pad 2: Net-(U3-GND) -> Net-(U1-GND)
- R3 pad 1: Net-(U4-VO) -> +3.3V
- R3 pad 2: Net-(U4-GND) -> Net-(U2-GND)
- R4 pad 1: Net-(U3-GND) -> +3.3V
- R4 pad 2: GND -> Net-(D1-A)
- R5 pad 1: Net-(U4-GND) -> Net-(U1-GND)
- R6 pad 1: Net-(J4-Pad2) -> Net-(U2-GND)
- R6 pad 2: Net-(U9A-+) -> GND
- R7 pad 1: Net-(U9A-+) -> Net-(R7-Pad1)
- R7 pad 2: GND -> /gpio/TEST_BUTTON
- R8 pad 1: +5VD -> Net-(D8-A)
- R8 pad 2: Net-(U9C-+) -> /gpio/TEST_LED
- R9 pad 1: Net-(U9C-+) -> Net-(C25-Pad2)
- RV1 pad 2: Net-(U6-VE) -> Net-(DS1-V0)
- RV2 pad 1: /gpio/SPKR -> +5V
- RV2 pad 2: Net-(U8-+) -> Net-(DS1-PadA)
- SW1 pad 2: Net-(U2-MR) -> Net-(U3-MR)
- TP1 pad 1: +3.3V -> /gpio/TEST_BUTTON
- TP2 pad 1: GND -> /gpio/TEST_LED
- TP3 pad 1: /gpio/TEST -> +3.3V
- U1 pad 1: Net-(U1-RF_P) -> Net-(U1-GND)
- U1 pad 2: Net-(U1-RF_N) -> +5V
- U1 pad 3: Net-(U1-X32K_Q1) -> +VBAT
- U2 pad 1: unconnected-(U2-GND-Pad1) -> Net-(U2-GND)
- U2 pad 2: unconnected-(U2-GND-Pad2) -> +3.3V
- U2 pad 3: Net-(J2-~{SRST}) -> +5V
- U3 pad 1: Net-(U3-GND) -> GND
- U3 pad 2: +5V -> GND
- U3 pad 3: +5VD -> Net-(J2-~{SRST})
- U4 pad 1: Net-(U4-GND) -> /RF_P
- U4 pad 2: Net-(U4-VO) -> /RF_N
- U4 pad 3: +5V -> Net-(U4-X32K_Q1)
- U5 pad 12: Net-(D6-K) -> Net-(D7-K)
- U5 pad 13: Net-(D5-K) -> Net-(D6-K)
- U5 pad 14: Net-(D4-K) -> Net-(D5-K)
- U5 pad 15: Net-(D3-K) -> Net-(D4-K)
- U5 pad 16: +5V -> +3.3V
- U5 pad 6: +5V -> +3.3V
- U6 pad 1: GND -> /gpio/LCD_RW
- U6 pad 10: Net-(U6-D3) -> GND
- U6 pad 11: Net-(U6-D4) -> /gpio/LCD_DATA7
- U6 pad 12: Net-(U6-D5) -> /gpio/LCD_DATA6
- U6 pad 13: Net-(U6-D6) -> /gpio/LCD_DATA5
- U6 pad 14: Net-(U6-D7) -> /gpio/LCD_DATA4
- U6 pad 2: +5V -> Net-(DS1-DB7)
- U6 pad 3: Net-(U6-VE) -> Net-(DS1-DB6)
- U6 pad 4: /gpio/LCD_RS -> Net-(DS1-DB5)
- U6 pad 5: /gpio/LCD_RW -> Net-(DS1-DB4)
- U6 pad 6: /gpio/LCD_E -> Net-(DS1-DB3)
- U6 pad 7: Net-(U6-D0) -> Net-(DS1-DB2)
- U6 pad 8: Net-(U6-D1) -> Net-(DS1-DB1)
- U6 pad 9: Net-(U6-D2) -> Net-(DS1-DB0)
- U7 pad 1: /gpio/LCD_RW -> Net-(C26-Pad1)
- U7 pad 2: Net-(U6-D0) -> GND
- U7 pad 3: Net-(U6-D1) -> Net-(U7-+)
- U7 pad 4: Net-(U6-D2) -> GND
- U7 pad 5: Net-(U6-D3) -> Net-(C24-Pad1)
- U7 pad 6: Net-(U6-D4) -> +5V
- U7 pad 7: Net-(U6-D5) -> Net-(U7-BYPASS)
- U7 pad 8: Net-(U6-D6) -> Net-(C26-Pad2)
- U8 pad 1: Net-(C28-Pad1) -> /gpio/SERVO2_POS
- U8 pad 2: GND -> /gpio/SERVO2_POS
- U8 pad 3: Net-(U8-+) -> Net-(U8A-+)
- U8 pad 4: GND -> +3.3V
- U8 pad 5: Net-(C27-Pad1) -> Net-(U8B-+)
- U8 pad 6: +5V -> /gpio/SERVO1_POS
- U8 pad 7: Net-(U8-BYPASS) -> /gpio/SERVO1_POS
- U8 pad 8: Net-(C28-Pad2) -> /gpio/VBAT_READ
- U9 pad 1: /gpio/SERVO1_POS -> +3.3V
- U9 pad 10: Net-(U9C-+) -> Net-(U9-REGOUT)
- U9 pad 11: GND -> unconnected-(U9-FSYNC-Pad11)
- U9 pad 13: unconnected-(U9D---Pad13) -> +3.3V
- U9 pad 14: unconnected-(U9-Pad14) -> (no net)
- U9 pad 2: /gpio/SERVO1_POS -> (no net)
- U9 pad 3: Net-(U9A-+) -> (no net)
- U9 pad 4: +3.3V -> (no net)
- U9 pad 5: Net-(U9B-+) -> (no net)
- U9 pad 6: /gpio/SERVO2_POS -> (no net)
- U9 pad 7: /gpio/SERVO2_POS -> unconnected-(U9-AUX_CL-Pad7)
- U9 pad 8: /gpio/VBAT_READ -> +3.3V
- U9 pad 9: /gpio/VBAT_READ -> /gpio/SPI_MISO
- X1 pad 1: Net-(U1-X48M_N) -> Net-(U4-X48M_N)
- X1 pad 3: Net-(U1-X48M_P) -> Net-(U4-X48M_P)
- X2 pad 1: Net-(U1-X32K_Q2) -> Net-(U4-X32K_Q2)
- X2 pad 2: Net-(U1-X32K_Q1) -> Net-(U4-X32K_Q1)
Routing:
- net +3.3V: track 0.00 -> 350.3 mm, vias 0 -> 16
- net GND: track 0.00 -> 249.4 mm, vias 0 -> 101
- net +5V: track 0.00 -> 236.5 mm, vias 0 -> 5
- net +VBAT: track 0.00 -> 156.2 mm
- net /gpio/SERVO2_PWM: track 0.00 -> 95.4 mm, vias 0 -> 1
- net /gpio/KEYPAD_ROWB: track 0.00 -> 94.8 mm, vias 0 -> 4
- net /gpio/TEST_LED: track 0.00 -> 94.1 mm, vias 0 -> 6
- net /gpio/KEYPAD_COL1: track 0.00 -> 93.5 mm, vias 0 -> 2
- net /gpio/KEYPAD_COL2: track 0.00 -> 92.6 mm, vias 0 -> 2
- net /gpio/KEYPAD_COL4: track 0.00 -> 92.0 mm, vias 0 -> 2
- net /gpio/KEYPAD_COL3: track 0.00 -> 91.8 mm, vias 0 -> 2
- net /gpio/LCD_RW: track 0.00 -> 90.6 mm, vias 0 -> 1
- net /gpio/TEST: track 0.00 -> 88.7 mm, vias 0 -> 6
- net /gpio/TEST_BUTTON: track 0.00 -> 87.7 mm, vias 0 -> 4
- net /gpio/KEYPAD_ROWA: track 0.00 -> 87.6 mm, vias 0 -> 2
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- added copper zone on B.Cu, net GND
- added copper zone on F.Cu, net GND
Other:
- board size 104.1 x 144.8 mm -> 98 x 150 mm
- rule solder_mask_min_width: 0.125 -> 0.13
- board text added: "Backlight"
- board text added: "Contrast"
- board text added: "EE 110 Alpha Board Adam Krivka March 2024"
- board text added: "Features: - Bluetooth - LCD - Keypad - Speaker - SD card - Servo control - IMU"
- board text added: "GND"
- board text added: "V+"
- board text added: "Volume"

Commit message: Ilana committing from laptop
Parts:
- added ?: , , F.Cu at (90.9, 59.2)
- added ?: , , F.Cu at (80.0, 91.7)
- added ?: , , F.Cu at (108.2, 139.4)
- added D10: D_Small_Filled, Diode_SMD:D_1206_3216Metric_Pad1.42x1.75mm_HandSolder, F.Cu at (113.8, 146.8)
- added D11: D_Small_Filled, Diode_SMD:D_1206_3216Metric_Pad1.42x1.75mm_HandSolder, F.Cu at (114.0, 162.1)
- added D9: LED_BLUE, LED_SMD:LED_0603_1608Metric_Pad1.05x0.95mm_HandSolder, F.Cu at (48.5, 154.4)
- added R8: 200, Resistor_SMD:R_0603_1608Metric_Pad0.98x0.95mm_HandSolder, F.Cu at (55.6, 154.4)
- C1, C10, C11, C12, C14, C16, C2, C21, C3, C4, C5, C6, C7, C8, C9: footprint Capacitor_Tantalum_SMD:CP_EIA-1608-08_AVX-J -> Capacitor_Tantalum_SMD:CP_EIA-1608-08_AVX-J_Pad1.25x1.05mm_HandSolder
- C13, C15, C17, C18, C19, C20: footprint Capacitor_SMD:C_1206_3216Metric -> Capacitor_SMD:C_1206_3216Metric_Pad1.33x1.80mm_HandSolder
- C22, C23, C24, C25, C26, C27, C28, C29: footprint Capacitor_SMD:C_0603_1608Metric -> Capacitor_SMD:C_0603_1608Metric_Pad1.08x0.95mm_HandSolder
- D1: value POWER LED -> LED
- D2, D3, D4, D5, D6, D7: footprint Diode_SMD:D_0603_1608Metric -> Diode_SMD:D_0603_1608Metric_Pad1.05x0.95mm_HandSolder
- D8: value TEST_LED -> LED_GREEN; footprint LED_SMD:LED_0603_1608Metric -> LED_SMD:LED_0603_1608Metric_Pad1.05x0.95mm_HandSolder
- J5: value Servo1 -> 4P4C
- J6: value Servo2 -> 4P4C
- L2: footprint Inductor_SMD:L_0603_1608Metric -> Inductor_SMD:L_0603_1608Metric_Pad1.05x0.95mm_HandSolder
- L3, L4, L5: footprint Inductor_SMD:L_1206_3216Metric -> Inductor_SMD:L_1206_3216Metric_Pad1.22x1.90mm_HandSolder
- R1: renamed from R7; footprint Resistor_SMD:R_0603_1608Metric -> Resistor_SMD:R_0603_1608Metric_Pad0.98x0.95mm_HandSolder
- R10, R11, R12, R13, R14, R15, R2, R3, R4, R5, R6, R9: footprint Resistor_SMD:R_0603_1608Metric -> Resistor_SMD:R_0603_1608Metric_Pad0.98x0.95mm_HandSolder
- R7: renamed from R8; footprint Resistor_SMD:R_0603_1608Metric -> Resistor_SMD:R_0603_1608Metric_Pad0.98x0.95mm_HandSolder
- RV2: value 10k -> 1k
- TP2: value TEST_LED -> TEST_GREEN
- TP3: renamed from TP5; value TEST -> TEST_BLUE
- U9: footprint Sensor_Motion:InvenSense_QFN-24_3x3mm_P0.4mm -> Package_DFN_QFN:QFN-24-1EP_3x3mm_P0.4mm_EP1.75x1.6mm
- moved TP3 9.37 mm to (60.7, 154.4)
- moved TP5 7.85 mm to (66.7, 151.1)
- moved D2 5.33 mm to (86.4, 104.9)
- moved D3 4.85 mm to (82.0, 99.8)
- moved J2 3.81 mm to (75.7, 103.6)
- moved R11 2.76 mm to (112.7, 137.2)
- moved R15 2.76 mm to (124.7, 137.9)
- moved R10 2.76 mm to (111.2, 134.6)
- moved R12 2.76 mm to (124.6, 134.6)
- moved R13 2.76 mm to (124.6, 131.8)
- moved R14 2.76 mm to (124.6, 140.7)
- moved U8 2.76 mm to (118.1, 135.9)
- moved J5 1.14 mm to (121.3, 154.3)
- moved R2 1.02 mm to (84.3, 151.6)
- moved TP4 0.92 mm to (62.2, 136.7)
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- renumbered TP3 to TP4, TP4 to TP5
Connections:
- net /gpio/TEST renamed /gpio/TEST_BLUE
- net /gpio/TEST_LED renamed /gpio/TEST_GREEN
- J5 pad 4: +VBAT -> Net-(D10-K)
- J6 pad 4: +VBAT -> Net-(D11-K)
- R4 pad 1: +3.3V -> +5V
- U4 pad 38: /gpio/VBAT_READ -> /gpio/SPKR
- U4 pad 39: /gpio/SERVO2_POS -> /gpio/VBAT_READ
- U4 pad 40: /gpio/SERVO1_POS -> /gpio/SERVO2_POS
- U4 pad 41: /gpio/SERVO2_PWM -> /gpio/SERVO1_POS
- U4 pad 42: /gpio/SERVO1_PWM -> /gpio/SERVO2_PWM
- U4 pad 43: /gpio/SPKR -> /gpio/SERVO1_PWM
Routing:
- net GND: track 249.4 -> 892.3 mm, vias 101 -> 66
- net /gpio/SERVO2_POS: track 60.4 -> 88.6 mm, vias 0 -> 2
- net +3.3V: track 350.3 -> 324.6 mm, vias 16 -> 18
- net +VBAT: track 156.2 -> 133.7 mm
- net /gpio/VBAT_READ: track 51.8 -> 74.2 mm
- net /gpio/SERVO1_PWM: track 75.1 -> 95.8 mm
- net /gpio/SERVO1_POS: track 53.8 -> 73.0 mm
- net +5V: track 236.5 -> 251.5 mm
- net /gpio/SERVO2_PWM: track 95.4 -> 109.6 mm
- net /gpio/TEST_BUTTON: track 87.7 -> 76.2 mm
- net /gpio/SPKR: track 53.9 -> 45.3 mm
- net /gpio/TEST_GREEN: track 94.1 -> 85.6 mm, vias 6 -> 4
- net Net-(D10-K): track 0.00 -> 6.06 mm
- net Net-(D11-K): track 0.00 -> 5.86 mm
- net Net-(D9-A): track 0.00 -> 5.50 mm
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Other:
- rule pad_to_mask_clearance: 0.08 -> 0
- board text added: "EE 110 Alpha Board Adam Krivka v0.2"
- board text removed: "EE 110 Alpha Board Adam Krivka March 2024"
