File: alpha_board/hardware_old/ee110_alpha_board.kicad_sch (KiCad schematic)
At the start: 46 parts, among them J1 power, J2 AVR-JTAG-10, SW1 RESET, U1 LM1086, U2 LM1086, U3 LM372x, U4 CC2652R1FRGZR, X1 48MHz, X2 32.768KHz

Commit message: first revision
Parts:
- added R1: 1, Resistor_SMD:R_0603_1608Metric, symbol Device:R_US
- R3: renamed from R4; value 200 -> 470
- SW1: footprint Button_Switch_SMD:SW_SPST_TL3342 -> Button_Switch_THT:SW_PUSH_6mm
- renumbered R3 to R4
Connections:
- net gpio/TEST_BUTTON is gone; now on net gpio/TEST: U4.32 (DIO_22)
- net gpio/TEST_LED is gone; now on net gpio/VBAT_READ: U4.36 (DIO_23)
- net +3.3V: now also R1.2; no longer C3.1, R4.1, U2.2 (VO)
- net gpio/SERVO1_POS: now also U4.38 (DIO_25); no longer U4.40 (DIO_27)
- net gpio/SERVO1_PWM: now also U4.40 (DIO_27); no longer U4.42 (DIO_29)
- net gpio/SERVO2_POS: now also U4.37 (DIO_24); no longer U4.39 (DIO_26)
- net gpio/SERVO2_PWM: now also U4.39 (DIO_26); no longer U4.41 (DIO_28)
- net gpio/SPKR: now also U4.41 (DIO_28); no longer U4.43 (DIO_30)
- net gpio/TEST: no longer U4.37 (DIO_24)
- net gpio/VBAT_READ: no longer U4.38 (DIO_25)
- net +VBAT renamed +5VD
- new net: C3.1, R1.1, R4.1, U2.2 (VO)
Other:
- sheet gpio ports: added none; removed TEST_BUTTON, TEST_LED
- note removed: "power led"
Changed lines of the file:
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@@
 		(title "EE 110 Alpha Board")
 		(date "2024-02-05")
-		(rev "0.2")
+		(rev "0.1")
 		(company "Adam Krivka")
 	)
@@
 	)
 	(junction
-		(at 127 33.02)
-		(diameter 0)
-		(color 0 0 0 0)
-	)
-	(junction
 		(at 128.905 77.47)
 		(diameter 0)
@@
 	)
 	(junction
+		(at 117.475 33.02)
+		(diameter 0)
+		(color 0 0 0 0)
+	)
+	(junction
 		(at 126.365 146.05)
 		(diameter 0)
@@
 	)
 	(junction
+		(at 127 33.02)
+		(diameter 0)
+		(color 0 0 0 0)
+	)
+	(junction
 		(at 128.905 92.71)
 		(diameter 0)
@@
 		(color 0 0 0 0)
 	)
-	(junction
-		(at 117.475 33.02)
-		(diameter 0)
-		(color 0 0 0 0)
-	)
 	(wire
 		(pts
@@
 	(wire
 		(pts
-			(xy 108.585 33.02) (xy 117.475 33.02)
+			(xy 117.475 33.02) (xy 119.38 33.02)
 		)
 		(stroke
@@
 	(wire
 		(pts
-			(xy 117.475 33.02) (xy 127 33.02)
-		)
-		(stroke
-			(width 0)
-			(type default)
-		)
-	)
-	(wire
-		(pts
 			(xy 92.71 48.26) (xy 92.71 48.895)
 		)
@@
 	(wire
 		(pts
+			(xy 117.475 33.02) (xy 108.585 33.02)
+		)
+		(stroke
+			(width 0)
+			(type default)
+		)
+	)
+	(wire
+		(pts
 			(xy 221.615 48.26) (xy 211.455 48.26)
 		)
@@
 		(exclude_from_sim no)
 		(at 17.78 17.78 0)
-		(size 118.745 43.18)
+		(size 115.57 43.18)
 		(stroke
 			(width 0)
@@
 		)
 	)
-	(text "power led"
-		(exclude_from_sim no)
-		(at 130.175 50.165 0)
-		(effects
-			(font
-				(size 1.27 1.27)
-			)
-		)
-	)
 	(text "C_{T}=2uF"
 		(exclude_from_sim no)
@@
 		(on_board yes)
 		(dnp no)
-		(property "Reference" "#PWR030"
+		(property "Reference" "#PWR029"
 			(at 62.865 150.495 0)
 			(effects
@@
 			(project "ee110_alpha_board"
 				(path "/060641a7-5b01-4853-a128-70e9cd5157bc"
-					(reference "#PWR030")
+					(reference "#PWR029")
 					(unit 1)
 				)
@@
 		(on_board yes)
 		(dnp no)
+		(fields_autoplaced yes)
 		(property "Reference" "#PWR04"
 			(at 37.465 35.56 0)
@@
 			)
 		)
-		(property "Value" "+VBAT"
-			(at 36.83 27.94 0)
+		(property "Value" "+5VD"
+			(at 37.465 27.94 0)
 			(effects
 				(font
@@
 		(dnp no)
 		(fields_autoplaced yes)
-		(property "Reference" "R3"
+		(property "Reference" "R4"
 			(at 111.125 36.195 0)
 			(effects
@@
 			(project "ee110_alpha_board"
 				(path "/060641a7-5b01-4853-a128-70e9cd5157bc"
-					(reference "R3")
+					(reference "R4")
 					(unit 1)
 				)
@@
 		(on_board yes)
 		(dnp no)
-		(property "Reference" "#PWR031"
+		(property "Reference" "#PWR030"
 			(at 77.47 150.495 0)
 			(effects
@@
 			(project "ee110_alpha_board"
 				(path "/060641a7-5b01-4853-a128-70e9cd5157bc"
-					(reference "#PWR031")
+					(reference "#PWR030")
 					(unit 1)
 				)
@@
 			)
 		)
-		(property "Footprint" "Button_Switch_SMD:SW_SPST_TL3342"
+		(property "Footprint" "Button_Switch_THT:SW_PUSH_6mm"
 			(at 31.75 84.455 0)
 			(effects
@@
 		(dnp no)
 		(fields_autoplaced yes)
-		(property "Reference" "#PWR033"
+		(property "Reference" "#PWR032"
 			(at 120.015 157.48 0)
 			(effects
@@
 			(project "ee110_alpha_board"
 				(path "/060641a7-5b01-4853-a128-70e9cd5157bc"
-					(reference "#PWR033")
+					(reference "#PWR032")
 					(unit 1)
 				)
@@
 	)
 	(symbol
+		(lib_id "Device:R_US")
+		(at 123.19 33.02 90)
+		(unit 1)
+		(exclude_from_sim no)
+		(in_bom yes)
+		(on_board yes)
+		(dnp no)
+		(property "Reference" "R1"
+			(at 123.19 27.94 90)
+			(effects
+				(font
+					(size 1.27 1.27)
+				)
+			)
+		)
+		(property "Value" "1"
+			(at 123.19 30.48 90)
+			(effects
+				(font
+					(size 1.27 1.27)
+				)
+			)
+		)
+		(property "Footprint" "Resistor_SMD:R_0603_1608Metric"
+			(at 123.444 32.004 90)
+			(effects
+				(font
+					(size 1.27 1.27)
+				)
+				(hide yes)
+			)
+		)
+		(property "Datasheet" "~"
+			(at 123.19 33.02 0)
+			(effects
+				(font
+					(size 1.27 1.27)
+				)
+				(hide yes)
+			)
+		)
+		(property "Description" ""
+			(at 123.19 33.02 0)
+			(effects
+				(font
+					(size 1.27 1.27)
+				)
+				(hide yes)
+			)
+		)
+		(pin "2"
+		)
+		(pin "1"
+		)
+		(instances
+			(project "ee110_alpha_board"
+				(path "/060641a7-5b01-4853-a128-70e9cd5157bc"
+					(reference "R1")
+					(unit 1)
+				)
+			)
+		)
+	)
+	(symbol
 		(lib_id "Device:C_Polarized_Small_US")
 		(at 103.505 125.73 0)
@@
 		(dnp no)
 		(fields_autoplaced yes)
-		(property "Reference" "#PWR034"
+		(property "Reference" "#PWR033"
 			(at 201.93 167.005 0)
 			(effects
@@
 			(project "ee110_alpha_board"
 				(path "/060641a7-5b01-4853-a128-70e9cd5157bc"
-					(reference "#PWR034")
+					(reference "#PWR033")
 					(unit 1)
 				)
@@
 		(on_board yes)
 		(dnp no)
-		(property "Reference" "#PWR029"
+		(property "Reference" "#PWR028"
 			(at 48.26 150.495 0)
 			(effects
@@
 			(project "ee110_alpha_board"
 				(path "/060641a7-5b01-4853-a128-70e9cd5157bc"
-					(reference "#PWR029")
+					(reference "#PWR028")
 					(unit 1)
 				)
@@
 		(dnp no)
 		(fields_autoplaced yes)
-		(property "Reference" "#PWR028"
+		(property "Reference" "#PWR027"
 			(at 114.935 149.86 0)
 			(effects
@@
 			(project "ee110_alpha_board"
 				(path "/060641a7-5b01-4853-a128-70e9cd5157bc"
-					(reference "#PWR028")
+					(reference "#PWR027")
 					(unit 1)
 				)
@@
 		(dnp no)
 		(fields_autoplaced yes)
-		(property "Reference" "R4"
-			(at 129.54 35.5599 0)
+		(property "Reference" "R3"
+			(at 129.54 35.56 0)
 			(effects
 				(font
@@
 			)
 		)
-		(property "Value" "200"
-			(at 129.54 38.0999 0)
+		(property "Value" "470"
+			(at 129.54 38.1 0)
 			(effects
 				(font
@@
 			(project "ee110_alpha_board"
 				(path "/060641a7-5b01-4853-a128-70e9cd5157bc"
-					(reference "R4")
+					(reference "R3")
 					(unit 1)
 				)
@@
 		(on_board yes)
 		(dnp no)
-		(property "Reference" "#PWR032"
+		(property "Reference" "#PWR031"
 			(at 25.4 156.21 0)
 			(effects
@@
 			(project "ee110_alpha_board"
 				(path "/060641a7-5b01-4853-a128-70e9cd5157bc"
-					(reference "#PWR032")
+					(reference "#PWR031")
 					(unit 1)
 				)
@@
 		(on_board yes)
 		(dnp no)
-		(property "Reference" "#PWR027"
+		(property "Reference" "#PWR078"
 			(at 88.9 144.78 0)
 			(effects
@@
 			(project "ee110_alpha_board"
 				(path "/060641a7-5b01-4853-a128-70e9cd5157bc"
-					(reference "#PWR027")
+					(reference "#PWR078")
 					(unit 1)
 				)
@@
 		(dnp no)
 		(fields_autoplaced yes)
-		(property "Reference" "#PWR035"
+		(property "Reference" "#PWR034"
 			(at 144.145 168.91 0)
 			(effects
@@
 			(project "ee110_alpha_board"
 				(path "/060641a7-5b01-4853-a128-70e9cd5157bc"
-					(reference "#PWR035")
+					(reference "#PWR034")
 					(unit 1)
 				)
@@
 		)
 		(pin "SERVO1_PWM" bidirectional
-			(at 232.41 151.13 180)
+			(at 232.41 146.05 180)
 			(effects
 				(font
@@
 		)
 		(pin "SERVO2_PWM" bidirectional
-			(at 232.41 148.59 180)
+			(at 232.41 143.51 180)
 			(effects
 				(font
@@
 		)
 		(pin "SERVO1_POS" bidirectional
-			(at 232.41 146.05 180)
+			(at 232.41 140.97 180)
 			(effects
 				(font
@@
 		)
 		(pin "SERVO2_POS" bidirectional
-			(at 232.41 143.51 180)
+			(at 232.41 138.43 180)
 			(effects
 				(font
@@
 		)
 		(pin "VBAT_READ" bidirectional
-			(at 232.41 140.97 180)
+			(at 232.41 135.89 180)
 			(effects
 				(font
@@
 		)
 		(pin "SPKR" input
-			(at 232.41 153.67 180)
+			(at 232.41 148.59 180)
 			(effects
 				(font
@@
 		)
 		(pin "TEST" bidirectional
-			(at 232.41 138.43 180)
-			(effects
-				(font
-					(size 1.27 1.27)
-				)
-				(justify left)
-			)
-		)
-		(pin "TEST_BUTTON" bidirectional
 			(at 232.41 133.35 180)
 			(effects
 				(font
-					(size 1.27 1.27)
-				)
-				(justify left)
-			)
-		)
-		(pin "TEST_LED" bidirectional
-			(at 232.41 135.89 180)
-			(effects
-				(font
