File: alpha_board/hardware_old/ee110_alpha_board_gpio.kicad_sch (KiCad schematic)
At the start: 41 parts, among them J4 Micro_SD_Card, J5 4P4C, J6 4P4C, SW2 TEST_BUTTON, U5 74LS138, U6 74LVC245, U7 LM386, U8 LM2902, U9 MPU-9250

Commit message: first revision
Parts:
- removed D8: LED, LED_SMD:LED_0603_1608Metric, symbol Device:LED
- removed R7: 100, Resistor_SMD:R_0603_1608Metric, symbol Device:R_US
- removed R8: 200, Resistor_SMD:R_0603_1608Metric, symbol Device:R_US
- removed SW2: TEST_BUTTON, Button_Switch_SMD:SW_SPST_TL3342, symbol Switch:SW_Push
- removed TP1: TEST_BUTTON, TestPoint:TestPoint_THTPad_2.0x2.0mm_Drill1.0mm, symbol Connector:TestPoint
- removed TP2: TEST_LED, TestPoint:TestPoint_THTPad_2.0x2.0mm_Drill1.0mm, symbol Connector:TestPoint
- DS1: footprint My_Footprint:WINSTAR-WH1604A -> My_Footprint:LCD_LCD-20X4B
- RV2: renamed from RV3; footprint Potentiometer_THT:Potentiometer_Bourns_3296P_Horizontal -> My_Footprint:TRIM_PTV09A-2015U-B103
- renumbered R12 to R10, R13 to R11, R14 to R12, R15 to R13, R9 to R7, R10 to R8, R11 to R9, RV2 to RV3, TP3 to TP1, TP4 to TP2, TP5 to TP3, U9 to U10, U5 to U6, U6 to U7, U7 to U8, U8 to U9
Connections:
- net +3.3V: no longer U7.20 (VCC)
- net GND: now also DS1.16 (K), DS1.S1 (SHIELD), DS1.S2 (SHIELD), DS1.S3 (SHIELD), DS1.S4 (SHIELD); no longer DS1.K
- net at RV3.2: now also DS1.15 (A); no longer DS1.A
- net +VBAT renamed +5VD
- new net +3V3: U7.20 (VCC)
Other:
- moved on the sheet: TP1, TP2, TP3
