File: boards/alpha_board/pcb_rev2/ee110_alpha_board_rev2.kicad_sch (KiCad schematic)
At the start: 53 parts, among them J1 power, J2 Conn_ARM_JTAG_SWD_10, SW1 RESET, SW2 TEST_BUTTON, U1 TLV76150DCY, U2 TLV76133DCY, U3 NC7SZ08M5X, U4 LM3724EM5-4.63/NOPB, U5 CC2652, X1 48MHz, X2 32.768KHz

Commit message: split body-back, body-top and body-front into smaller parts
Parts:
- removed J1: power, Alpha Board rev2 library:My_Power_Connector, symbol Connector:Conn_01x02_Pin
- removed U3: NC7SZ08M5X, Package_TO_SOT_SMD:SOT-23-5_HandSoldering, symbol and_gate:NC7SZ08M5X
- added D1, D2: D_Small_Filled, Diode_SMD:D_SOD-323F, symbol Device:D_Small_Filled
- added J1: POWER, My_Footprint:1pin, symbol Connector:Conn_01x01_Pin
- added J3: GND, My_Footprint:1pin, symbol Connector:Conn_01x01_Pin
- added R1: 4.7k, Resistor_SMD:R_0805_2012Metric_Pad1.20x1.40mm_HandSolder, symbol Device:R_US
- D5: renamed from D3; footprint LED_SMD:LED_0805_2012Metric_Pad1.15x1.40mm_HandSolder -> LED_THT:LED_D3.0mm
- R5: renamed from R4; value 200 -> 280
- renumbered D1 to D3, D2 to D4, R1 to R2, R2 to R3, R3 to R4, U4 to U3, U5 to U4
Connections:
- net +3.3V: now also R1.1; no longer R5.1
- net +5V: now also R5.1
- net +VBAT: now also J1.1 (Pin_1)
- net GND: now also J3.1 (Pin_1)
- net at U4.35 (RESET_N): now also D1.2 (A), D2.2 (A), R1.2
- net at J2.10 (~{RESET}): now also D2.1 (K)
- net at U3.3 (RESET_N): now also D1.1 (K)
Other:
- moved on the sheet: JP1

Commit message: 4/27
Parts:
- removed D3: TEST_GREEN, LED_SMD:LED_0805_2012Metric_Pad1.15x1.40mm_HandSolder, symbol Device:LED
- removed D4: TEST_BLUE, LED_SMD:LED_0805_2012Metric_Pad1.15x1.40mm_HandSolder, symbol Device:LED
- removed D5: POWER_LED, LED_THT:LED_D3.0mm, symbol Device:LED
- removed R2: 100, Resistor_SMD:R_0805_2012Metric_Pad1.20x1.40mm_HandSolder, symbol Device:R_US
- removed R3, R4: 200, Resistor_SMD:R_0805_2012Metric_Pad1.20x1.40mm_HandSolder, symbol Device:R_US
- removed R5: 280, Resistor_SMD:R_0805_2012Metric_Pad1.20x1.40mm_HandSolder, symbol Device:R_US
- removed SW2: TEST_BUTTON, Button_Switch_SMD:SW_SPST_TL3342, symbol Switch:SW_Push
- removed TP1: DIO22, TestPoint:TestPoint_THTPad_2.0x2.0mm_Drill1.0mm, symbol Connector:TestPoint
- removed TP2: DIO23, TestPoint:TestPoint_THTPad_2.0x2.0mm_Drill1.0mm, symbol Connector:TestPoint
- removed TP3: DIO24, TestPoint:TestPoint_THTPad_2.0x2.0mm_Drill1.0mm, symbol Connector:TestPoint
- removed TP4: +3.3V, TestPoint:TestPoint_THTPad_2.0x2.0mm_Drill1.0mm, symbol Connector:TestPoint
- removed TP5: GND, TestPoint:TestPoint_THTPad_2.0x2.0mm_Drill1.0mm, symbol Connector:TestPoint
- added SW3: SW_SPDT, Alpha Board rev2 library:EG1903, symbol Switch:SW_SPDT
Connections:
- net gpio/SERVO1_POS: now also U4.39 (DIO_26); no longer U4.41 (DIO_28)
- net gpio/SERVO1_PWM: now also U4.41 (DIO_28); no longer U4.43 (DIO_30)
- net gpio/SPKR: now also U4.43 (DIO_30); no longer U4.38 (DIO_25)
- net gpio/VBAT_READ: now also U4.38 (DIO_25); no longer U4.39 (DIO_26)
- net at B1.3: now also SW3.1 (A); no longer B1.1
- new net: B1.1, SW3.2 (B)
- no-connect marks 0 -> 1
